File: pcb/Microcontroller Lab Summer 2026/ESP+Power_Only/ESP+Power_Only.kicad_pcb (KiCad board)
At the start: 2 copper layers, 55.2 x 137.2 mm, 35 parts, among them J2 Power OUT, J3 SR_QH_Return, J4 Signals OUT, SW1 SW_Push, SW2 SW_Push, SW3 SW_Push, SW4 SW_Push, SW5 SW_SPDT, U1 TLV62568DBVR, U2 SN74AHCT125N, U4 TLV61048DBVR

Commit message: fixed PCB footprints, pending final review before order
Parts:
- C1, C4: footprint Capacitor_SMD:C_01005_0402Metric -> Capacitor_SMD:C_0402_1005Metric
- C2, C3, C5, C6, C7: footprint Capacitor_SMD:C_0201_0603Metric -> Capacitor_SMD:C_0603_1608Metric
- R11, R6: footprint Resistor_SMD:R_01005_0402Metric -> Resistor_SMD:R_0402_1005Metric
- R14, R9: footprint Resistor_SMD:R_0201_0603Metric -> Resistor_SMD:R_0603_1608Metric
- moved C3 5.83 mm to (96.1, 53.8), turned to 180 degrees
- moved C7 5.67 mm to (82.8, 44.5), turned to 180 degrees
- moved R7 0.81 mm to (78.1, 40.6)
- moved C4 0.76 mm to (121.0, 85.3)
- moved R11 0.61 mm to (94.0, 48.7)
- moved C5 0.50 mm to (121.5, 84.0)
- moved R6 0.41 mm to (78.0, 36.7)
- moved C1 0.32 mm to (121.8, 122.6)
- moved C2 0.21 mm to (77.3, 33.4)
- moved C6 0.14 mm to (92.5, 49.5)
Routing:
- net GND: track 24.1 -> 35.4 mm, vias 171 -> 153
- net +BATT: track 55.6 -> 45.8 mm
- net +3.3V: track 226.4 -> 223.9 mm
- net Net-(U4-FB): track 6.34 -> 5.80 mm

Commit message: fixed thermal relief areas, double checked new footprints, ready to order, need to generate gerber files, bom, placement csv and such
Parts:
- moved C5 0.40 mm to (121.5, 83.6)
Changed lines of the file:
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@@
 	(footprint "Capacitor_SMD:C_0603_1608Metric"
 		(layer "F.Cu")
-		(at 121.5 84 180)
+		(at 121.5 83.6 180)
 		(descr "Capacitor SMD 0603 (1608 Metric), square (rectangular) end terminal, IPC-7351 nominal, (Body size source: IPC-SM-782 page 76, https://www.pcb-3d.com/wordpress/wp-content/uploads/ipc-sm-782a_amendment_1_and_2.pdf)")
 		(tags "capacitor")
@@
 	)
 	(segment
-		(start 120.816919 134.85)
+		(start 120.5 123.483081)
+		(end 120.816919 123.8)
+		(width 0.2)
+		(layer "F.Cu")
+		(net "/LED_DATA_3.3V")
+	)
+	(segment
+		(start 120.816919 122.5)
 		(end 120.816919 121.1)
 		(width 0.2)
@@
 	)
 	(segment
+		(start 120.8 122.5)
+		(end 120.5 122.8)
+		(width 0.2)
+		(layer "F.Cu")
+		(net "/LED_DATA_3.3V")
+	)
+	(segment
+		(start 120.5 122.8)
+		(end 120.5 123.483081)
+		(width 0.2)
+		(layer "F.Cu")
+		(net "/LED_DATA_3.3V")
+	)
+	(segment
 		(start 76.516919 136.7)
 		(end 118.966919 136.7)
@@
 	)
 	(segment
+		(start 120.816919 122.5)
+		(end 120.8 122.5)
+		(width 0.2)
+		(layer "F.Cu")
+		(net "/LED_DATA_3.3V")
+	)
+	(segment
 		(start 118.966919 136.7)
 		(end 120.816919 134.85)
 		(width 0.2)
 		(layer "F.Cu")
+		(net "/LED_DATA_3.3V")
+	)
+	(segment
+		(start 120.816919 134.85)
+		(end 120.816919 123.8)
+		(width 0.2)
+		(layer "F.Cu")

Commit message: fixed detection pcb dip-16 footprint. fixed esp pcb charger board polarity, minor trace adjustments, level shifting for spi sclk and shift register mode signals. fixed charger board polarity footprint. last fix remaining is to get a more precise measurement for the two front pins on the charger board and update accordingly
Parts:
- J4: footprint Connector_PinHeader_2.54mm:PinHeader_1x04_P2.54mm_Vertical -> Connector_PinHeader_2.54mm:PinHeader_1x03_P2.54mm_Vertical
- moved C5 34.9 mm to (86.6, 83.9), turned to 0 degrees
- moved C4 34.1 mm to (86.9, 85.4), turned to 0 degrees
- moved J4 0.78 mm to (78.5, 85.3), turned to 0 degrees
Connections:
- J1 pad 15: +3.3V -> unconnected-(J1-VIN-Pad15)
- J1 pad 22: /SPI_SCLK -> /SPI_SCLK_3.3V
- J1 pad 23: /SR_LOAD -> /SR_LOAD_3.3V
- J1 pad 30: unconnected-(J1-3.3V-Pad30) -> +3.3V
- J4 pad 2: /SR_QH -> /SPI_SCLK_5V
- J4 pad 3: /SPI_SCLK -> /SR_LOAD_5V
- U2 pad 10: unconnected-(U2-*3OE-Pad10) -> GND
- U2 pad 4: unconnected-(U2-*2OE-Pad4) -> GND
- U2 pad 5: unconnected-(U2-2A-Pad5) -> /SPI_SCLK_3.3V
- U2 pad 6: unconnected-(U2-2Y-Pad6) -> /SPI_SCLK_5V
- U2 pad 8: unconnected-(U2-3Y-Pad8) -> /SR_LOAD_5V
- U2 pad 9: unconnected-(U2-3A-Pad9) -> /SR_LOAD_3.3V
Routing:
- net +3.3V: track 223.9 -> 310.3 mm, vias 0 -> 6
- net /SR_LOAD_5V: track 0.00 -> 62.5 mm, vias 0 -> 4
- net /SPI_SCLK_5V: track 0.00 -> 50.9 mm, vias 0 -> 4
- net /SPI_SCLK_3.3V: track 0.00 -> 41.7 mm, vias 0 -> 6
- net /SR_LOAD_3.3V: track 0.00 -> 40.2 mm, vias 0 -> 2
- net /SR_LOAD: track 30.1 -> 0.00 mm
- net /SPI_SCLK: track 30.1 -> 0.00 mm
- net GND: track 35.4 -> 33.7 mm, vias 153 -> 152
- net /LED_DATA_5V: track 42.3 -> 43.1 mm
