File: pcb/Microcontroller Lab Summer 2026/Sensors+LEDs/Sensors+LEDs.kicad_pcb (KiCad board)
At the start: 2 copper layers, 57.1 x 456.8 mm, 41 parts, among them J1 SR_QH_Return, J2 Signals_OUT, J3 Signals_IN, J4 Power_IN, J5 Power_OUT, U1 A3144, U2 A3144, U3 A3144, U4 SN74HC165N, U5 A3144, U6 A3144, U7 A3144, U8 A3144, U9 A3144

Commit message: fixed PCB footprints, pending final review before order
Parts:
- C1, C2, C3, C4, C5, C6, C7, C8, C9: footprint Capacitor_SMD:C_01005_0402Metric -> Capacitor_SMD:C_0402_1005Metric
- moved C8 0.36 mm to (-31.4, -218.7)
- moved C1 0.13 mm to (-31.3, 180.9)
- moved C2 0.10 mm to (-31.2, 123.9)
- moved C4 0.10 mm to (-31.2, 9.60)
- moved C5 0.10 mm to (-31.2, -47.5)
- moved C3 0.10 mm to (-31.2, 66.7)
- moved C6 0.08 mm to (-31.2, -104.6)
- moved C7 0.08 mm to (-31.2, -161.7)
Routing:
- net +5V: track 723.1 -> 727.5 mm

Commit message: fixed thermal relief areas, double checked new footprints, ready to order, need to generate gerber files, bom, placement csv and such
Changed lines of the file:
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@@
 			(at 0 -1.16 0)
 			(layer "F.SilkS")
+			(hide yes)
 			(effects
 				(font
@@
 			(at 0 1.16 0)
 			(layer "F.Fab")
+			(hide yes)
 			(effects
 				(font
@@
 			(at 0 -1.16 0)
 			(layer "F.SilkS")
+			(hide yes)
 			(effects
 				(font
@@
 			(at 0 1.16 0)
 			(layer "F.Fab")
+			(hide yes)
 			(effects
 				(font
@@
 			(at 0 -1.16 0)
 			(layer "F.SilkS")
+			(hide yes)
 			(effects
 				(font
@@
 			(at 0 1.16 0)
 			(layer "F.Fab")
+			(hide yes)
 			(effects
 				(font
@@
 			(at 0 -1.16 0)
 			(layer "F.SilkS")
+			(hide yes)
 			(effects
 				(font
@@
 			(at 0 1.16 0)
 			(layer "F.Fab")
+			(hide yes)
 			(effects
 				(font
@@
 			(at 0 -1.16 0)
 			(layer "F.SilkS")
+			(hide yes)
 			(effects
 				(font
@@
 			(at 0 1.16 0)
 			(layer "F.Fab")
+			(hide yes)
 			(effects
 				(font
@@
 			(at 0 -1.16 0)
 			(layer "F.SilkS")
+			(hide yes)
 			(effects
 				(font
@@
 			(at 0 1.16 0)
 			(layer "F.Fab")
+			(hide yes)
 			(effects
 				(font
@@
 			(at 0 -1.16 90)
 			(layer "F.SilkS")
+			(hide yes)
 			(effects
 				(font
@@
 			(at 0 1.16 90)
 			(layer "F.Fab")
+			(hide yes)
 			(effects
 				(font
@@
 			(at 0 -1.16 0)
 			(layer "F.SilkS")
+			(hide yes)
 			(effects
 				(font
@@
 			(at 0 1.16 0)
 			(layer "F.Fab")
+			(hide yes)
 			(effects
 				(font
@@
 			(at 0 -1.16 0)
 			(layer "F.SilkS")
+			(hide yes)
 			(effects
 				(font
@@
 			(at 0 1.16 0)
 			(layer "F.Fab")
+			(hide yes)
 			(effects
 				(font

Commit message: fixed detection pcb dip-16 footprint. fixed esp pcb charger board polarity, minor trace adjustments, level shifting for spi sclk and shift register mode signals. fixed charger board polarity footprint. last fix remaining is to get a more precise measurement for the two front pins on the charger board and update accordingly
Parts:
- U4: footprint Package_DIP:DIP-16_W10.16mm_LongPads -> Package_DIP:DIP-16_W7.62mm_LongPads
- moved R10 4.30 mm to (-53.3, -8.10)
- moved C9 2.22 mm to (-55.4, 6.27)
Routing:
- net /HE_D: track 28.9 -> 31.4 mm
- net /HE_C: track 90.1 -> 92.6 mm
- net /HE_B: track 151.1 -> 153.7 mm
- net /HE_A: track 212.9 -> 215.5 mm
- net +5V: track 727.5 -> 730.0 mm
- net /SR_QH_IN: track 233.4 -> 231.4 mm
- net /SR_QH_OUT: track 278.3 -> 276.4 mm
- net GND: vias 489 -> 490
