File: pcb/Microcontroller Lab Summer 2026/Sensors+LEDs/Sensors+LEDs.kicad_sch (KiCad schematic)
At the start: 41 parts, among them J1 SR_QH_Return, J2 Signals_OUT, J3 Signals_IN, J4 Power_IN, J5 Power_OUT, U1 A3144, U2 A3144, U3 A3144, U4 SN74HC165N, U5 A3144, U6 A3144, U7 A3144, U8 A3144, U9 A3144

Commit message: fixed PCB footprints, pending final review before order
Parts:
- C1, C2, C3, C4, C5, C6, C7, C8, C9: footprint Capacitor_SMD:C_01005_0402Metric -> Capacitor_SMD:C_0402_1005Metric
Changed lines of the file:
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@@
 			)
 		)
-		(property "Footprint" "Capacitor_SMD:C_01005_0402Metric"
+		(property "Footprint" "Capacitor_SMD:C_0402_1005Metric"
 			(at 27.94 48.5648 0)
 			(hide yes)
@@
 			)
 		)
-		(property "Footprint" "Capacitor_SMD:C_01005_0402Metric"
+		(property "Footprint" "Capacitor_SMD:C_0402_1005Metric"
 			(at 244.8052 139.7 0)
 			(hide yes)
@@
 			)
 		)
-		(property "Footprint" "Capacitor_SMD:C_01005_0402Metric"
+		(property "Footprint" "Capacitor_SMD:C_0402_1005Metric"
 			(at 27.94 178.1048 0)
 			(hide yes)
@@
 			)
 		)
-		(property "Footprint" "Capacitor_SMD:C_01005_0402Metric"
+		(property "Footprint" "Capacitor_SMD:C_0402_1005Metric"
 			(at 27.94 91.7448 0)
 			(hide yes)
@@
 			)
 		)
-		(property "Footprint" "Capacitor_SMD:C_01005_0402Metric"
+		(property "Footprint" "Capacitor_SMD:C_0402_1005Metric"
 			(at 27.94 156.5148 0)
 			(hide yes)
@@
 			)
 		)
-		(property "Footprint" "Capacitor_SMD:C_01005_0402Metric"
+		(property "Footprint" "Capacitor_SMD:C_0402_1005Metric"
 			(at 27.94 134.9248 0)
 			(hide yes)
@@
 			)
 		)
-		(property "Footprint" "Capacitor_SMD:C_01005_0402Metric"
+		(property "Footprint" "Capacitor_SMD:C_0402_1005Metric"
 			(at 27.94 113.3348 0)
 			(hide yes)
@@
 			)
 		)
-		(property "Footprint" "Capacitor_SMD:C_01005_0402Metric"
+		(property "Footprint" "Capacitor_SMD:C_0402_1005Metric"
 			(at 27.94 26.9748 0)
 			(hide yes)
@@
 			)
 		)
-		(property "Footprint" "Capacitor_SMD:C_01005_0402Metric"
+		(property "Footprint" "Capacitor_SMD:C_0402_1005Metric"
 			(at 27.94 70.1548 0)
 			(hide yes)

Commit message: fixed detection pcb dip-16 footprint. fixed esp pcb charger board polarity, minor trace adjustments, level shifting for spi sclk and shift register mode signals. fixed charger board polarity footprint. last fix remaining is to get a more precise measurement for the two front pins on the charger board and update accordingly
Parts:
- U4: footprint Package_DIP:DIP-16_W10.16mm_LongPads -> Package_DIP:DIP-16_W7.62mm_LongPads
Changed lines of the file:
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@@
 			)
 		)
-		(property "Footprint" "Package_DIP:DIP-16_W10.16mm_LongPads"
+		(property "Footprint" "Package_DIP:DIP-16_W7.62mm_LongPads"
 			(at 168.91 137.16 0)
 			(hide yes)
